File: hw/freewatch_v1/freewatch_v1.kicad_pcb (KiCad board)
At the start: 4 copper layers, 40 x 40 mm, 111 parts, among them P1 USB-MICRO-AB, P3 CONN_2, P6 CONN_2, P7 CONN_6, Q1 BSS138, Q2 BSS138, SW1 SW_PUSH, SW2 SW_PUSH, SW3 SW_PUSH, SW4 SW_PUSH, U1 PRTR5V0U2X, U10 MAX44009, U11 LSM303C, U12 MS5806-02BA, U13 ADP198, U14 LS013B7DH03, U15 EFM32GG330, U2 bq24072, U3 TPS780180300, U4 MAX17047, U5 TPS780180300, U6 M10478-A1, U7 MICRO_SDCARD_SPI, U8 ADP198, X1 32.768kHz, X2 48MHz

Commit message: hw: Move 1.8V LDO and motor to battery charger output (instead of 3V). Add pull-up on light sensor INT output. Add 10uF capacitor before motor switch.
Parts:
- C46, R26: moved to F.Cu
- SP1: moved to B.Cu
- moved SP1 5.58 mm to (119.7, 106.6)
- moved R26 1.39 mm to (123.5, 107.8)
- moved C46 1.38 mm to (123.5, 104.7)
Routing:
- net GND: track 258.9 -> 294.7 mm, vias 83 -> 93
- net /MCU_DISPLAY/SWDO: track 46.9 -> 44.2 mm
- net /MCU_DISPLAY/SWCLK: track 49.9 -> 47.5 mm
- net /MCU_DISPLAY/SW_BR: track 19.6 -> 22.1 mm, vias 2 -> 3
- net LS_INT_N: track 34.1 -> 31.9 mm
- net SD_EN: track 33.2 -> 31.1 mm
- net /MCU_DISPLAY/SWDIO: track 47.0 -> 45.0 mm
- net /MCU_DISPLAY/BUZ: track 12.6 -> 11.5 mm, vias 1 -> 2
- net BC_PGOOD_N: track 31.5 -> 32.0 mm
Other:
- board text added: "Licensed under CERN OHL v.1.2"
