File: hw/freewatch_v1/freewatch_v1.kicad_pcb (KiCad board)
At the start: 4 copper layers, 40 x 40 mm, 104 parts, among them P1 USB-MICRO-AB, P3 CONN_2, P6 CONN_2, P7 CONN_6, SW1 SW_PUSH, SW2 SW_PUSH, SW3 SW_PUSH, SW4 SW_PUSH, U1 PRTR5V0U2X, U10 MAX44009, U11 LSM303C, U12 MS5806-02BA, U13 ADP198, U14 LS013B7DH03, U15 EFM32GG330, U2 bq24072, U3 TPS780180300, U4 MAX17047, U5 MAX2659, U6 L70, U7 MICRO_SDCARD_SPI, U8 ADP198, U9 ADP198, X1 CRYSTAL_SMD

Commit message: Updated schematic files
Parts:
- removed ANT1: W3011A, freewatch_footprints:ANTENNA_W3011A
- removed D1, D2: CDBU0130R, freewatch_footprints:d_0603
- added C24: 10pF, Capacitors_SMD:c_0603, B.Cu at (106.0, 100.4)
- added C26: 10uF, Capacitors_SMD:c_0603, F.Cu at (123.8, 91.0)
- added C47: 100nF, Capacitors_SMD:c_0603, F.Cu at (106.4, 93.1)
- added HOLE_1.1MM: VAL**, freewatch_footprints:HOLE_1.1MM, F.Cu at (88.3, 112.3)
- added HOLE_1.1MM: VAL**, freewatch_footprints:HOLE_1.1MM, F.Cu at (124.3, 112.3)
- added HOLE_1.1MM: VAL**, freewatch_footprints:HOLE_1.1MM, F.Cu at (124.3, 76.3)
- added HOLE_1.1MM: VAL**, freewatch_footprints:HOLE_1.1MM, F.Cu at (88.3, 76.3)
- added L1: IND, Capacitors_SMD:c_0402, F.Cu at (99.9, 79.5)
- added Q1: BSS138, Transistors_SMD:sot23, F.Cu at (117.1, 84.8)
- added Q2: BSS138, Transistors_SMD:sot23, F.Cu at (117.2, 88.7)
- added R29: 10k, freewatch_footprints:r_0603, F.Cu at (114.5, 87.3)
- added R3: 10k, freewatch_footprints:r_0603, F.Cu at (110.0, 91.8)
- added R30: 10k, freewatch_footprints:r_0603, F.Cu at (119.6, 88.7)
- added R31: 100k, freewatch_footprints:r_0603, F.Cu at (116.5, 105.8)
- added X2: 48MHz, freewatch_footprints:ABM11_CRYSTAL, B.Cu at (108.0, 100.2)
- C1, C2, C3, C4, C5, C6, C7, C8, R4, R5, R6, R8, R9, U2, U3, U4: moved to F.Cu
- C10, C11: footprint Capacitors_SMD:c_0603 -> Capacitors_SMD:c_0402
- C12: value 100pF -> 22pF
- C13: value 33nF -> 22pF
- C15: value 10uF -> 2.2uF
- C16: value 100nF -> 22pF
- C18: value 100nF -> 10pF; moved to B.Cu
- C31, C32, C34, C36, C41, C42, C45, R25, R7, U15: moved to B.Cu
- C9: value 56pF -> 1uF
- P3: footprint freewatch_footprints:78171-0002 -> freewatch_footprints:SMD_BAT_CONN
- P6: footprint freewatch_footprints:78171-0002 -> freewatch_footprints:CONN_1MM_2P; moved to F.Cu
- P7: footprint freewatch_footprints:78171-5006 -> Connect:SIL-6
- R10: value 0 -> 10k
- R11, R12: value 100 -> 10k
- R13: value 470k -> 10k
- R14: value 4k7 -> 10R
- R17, R18, R19, R20: value 100k -> 91R
- R21, R22: footprint freewatch_footprints:r_0603 -> Capacitors_SMD:c_0402; moved to B.Cu
- SW1, SW2, SW3, SW4: value SW_PUSH -> EVQ-P4MB3K
- U5: value MAX2659 -> TPS780180300; footprint freewatch_footprints:UDFN6 -> freewatch_footprints:SON-6
- U6: value L70 -> M10478-A1; footprint freewatch_footprints:GPS_L70 -> freewatch_footprints:M10478-A1
- U9: value ADP198 -> SST25WF040B; footprint freewatch_footprints:LFCSP_8L -> freewatch_footprints:USON_2X3
- X1: value CRYSTAL_SMD -> 32.768kHz; moved to B.Cu
- moved R18 37.5 mm to (99.4, 98.9), turned to 90 degrees
- moved R19 35.4 mm to (98.5, 87.0), turned to 180 degrees
- moved D3 33.6 mm to (121.7, 84.0), turned to 270 degrees
- moved P6 32.9 mm to (119.8, 83.3), turned to 180 degrees
- moved C27 31.9 mm to (122.5, 86.2), turned to 0 degrees
- moved U13 29.2 mm to (122.5, 88.9), turned to 180 degrees
- moved C37 28.6 mm to (115.1, 92.2), turned to 180 degrees
- moved R9 28.0 mm to (96.0, 99.1)
- moved C14 26.7 mm to (106.3, 107.8)
- moved U8 26.5 mm to (108.6, 107.7)
- moved R13 26.2 mm to (114.5, 84.6), turned to 90 degrees
- moved C8 26.1 mm to (92.7, 100.4), turned to 270 degrees
- moved R12 25.9 mm to (119.6, 85.9)
- moved R14 25.7 mm to (123.8, 92.5)
- moved C6 25.7 mm to (91.4, 100.8), turned to 270 degrees
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Connections:
- C10 pad 1: Net-(ANT1-Pad1) -> Net-(C10-Pad1)
- C13 pad 1: Net-(C12-Pad1) -> GPS_RXD
- C15 pad 1: Net-(C15-Pad1) -> +1.8V
- C16 pad 1: Net-(C15-Pad1) -> +1.8V
- C17 pad 1: VCC -> +1.8V
- C18 pad 1: VCC -> Net-(C18-Pad1)
- C2 pad 1: Net-(C2-Pad1) -> +VIN
- C3 pad 1: Net-(C2-Pad1) -> +VIN
- C9 pad 1: Net-(C9-Pad1) -> +VIN
- C9 pad 2: Net-(C9-Pad2) -> GND
- R10 pad 1: Net-(ANT1-Pad1) -> Net-(R10-Pad1)
- R10 pad 2: Net-(C11-Pad1) -> +1.8V
- R11 pad 2: Net-(R11-Pad2) -> +1.8V
- R12 pad 1: Net-(C12-Pad1) -> GPS_TXD
- R12 pad 2: Net-(R12-Pad2) -> VCC
- R13 pad 1: Net-(D1-Pad1) -> Net-(C12-Pad1)
- R13 pad 2: VCC -> +1.8V
- R14 pad 1: USB_DM -> +VIN
- R14 pad 2: /MCU_DISPLAY/USB_DMPU -> Net-(C26-Pad1)
- U13 pad 7: VCC -> Net-(C26-Pad1)
- U13 pad 8: VCC -> Net-(C26-Pad1)
- U15 pad 1: SDA -> /MCU_DISPLAY/SW_TR
- U15 pad 10: /MCU_DISPLAY/LCD_EN -> /MCU_DISPLAY/LCD_VCC
- U15 pad 11: SD_MOSI -> /MCU_DISPLAY/LCD_DI
- U15 pad 12: SD_MISO -> SD_EN
- U15 pad 13: SD_CLK -> /MCU_DISPLAY/LCD_CLK
- U15 pad 14: SD_CS_N -> /MCU_DISPLAY/LCD_CS
- U15 pad 17: /MCU_DISPLAY/SW_TR -> /MCU_DISPLAY/SW_BR
- U15 pad 19: AC_INT_XL -> AC_INT_MAG
- U15 pad 2: SCL -> GPS_WAKUP
- U15 pad 21: AC_DRDY_MAG -> SDA
- U15 pad 22: AC_INT_MAG -> SCL
- U15 pad 24: Net-(U15-Pad24) -> Net-(C18-Pad1)
- U15 pad 28: AC_SDIO -> SD_MOSI
- U15 pad 29: AC_CS_XL -> SD_MISO
- U15 pad 3: FG_ALRT_N -> /MCU_DISPLAY/LCD_INV
- U15 pad 30: AC_CLK -> SD_CLK
- U15 pad 31: AC_CS_MAG -> SD_CS_N
- U15 pad 32: GPS_RXD -> AC_DRDY_MAG
- U15 pad 33: GPS_TXD -> AC_INT_XL
- U15 pad 34: SD_EN -> BC_CHG_N
- U15 pad 35: /MCU_DISPLAY/SW_TL -> BC_PGOOD_N
- U15 pad 36: GPS_PPS -> FG_ALRT_N
- U15 pad 37: GPS_STDBY -> /MCU_DISPLAY/SW_BL
- U15 pad 38: GPS_RST -> /MCU_DISPLAY/SW_TL
- U15 pad 4: /MCU_DISPLAY/SW_BR -> VM_EN
- U15 pad 41: GPS_EN -> AC_CS_XL
- U15 pad 42: /MCU_DISPLAY/SW_BL -> AC_CLK
- U15 pad 43: VM_EN -> AC_CS_MAG
- U15 pad 44: LS_INT_N -> AC_SDIO
- U15 pad 54: Net-(U15-Pad54) -> GPS_RST
- U15 pad 56: BC_CHG_N -> Net-(U15-Pad56)
- U15 pad 57: BC_PGOOD_N -> Net-(U15-Pad57)
- U15 pad 58: /MCU_DISPLAY/LCD_DI -> Net-(U15-Pad58)
- U15 pad 59: Net-(U15-Pad59) -> /MCU_DISPLAY/LCD_BKL2
- U15 pad 60: /MCU_DISPLAY/LCD_CLK -> /MCU_DISPLAY/LCD_BKL1
- U15 pad 61: /MCU_DISPLAY/LCD_CS -> GPS_ON_OFF
- U15 pad 62: /MCU_DISPLAY/LCD_INV -> GPS_RXD
- U15 pad 63: /MCU_DISPLAY/LCD_BKL1 -> GPS_TXD
- U15 pad 64: /MCU_DISPLAY/LCD_BKL2 -> Net-(U15-Pad64)
- U15 pad 7: Net-(U15-Pad7) -> LS_INT_N
- U15 pad 9: /MCU_DISPLAY/LCD_VCC -> /MCU_DISPLAY/LCD_EN
- U2 pad 10: Net-(C2-Pad1) -> +VIN
- U2 pad 11: Net-(C2-Pad1) -> +VIN
- U2 pad 5: Net-(C2-Pad1) -> +VIN
- U3 pad 4: Net-(C2-Pad1) -> +VIN
- U3 pad 6: Net-(C2-Pad1) -> +VIN
- U5 pad 1: GND -> +1.8V
- U5 pad 2: GND -> Net-(U5-Pad2)
- U5 pad 3: Net-(C11-Pad1) -> +VIN
- U5 pad 4: Net-(C12-Pad1) -> +VIN
- U5 pad 5: Net-(R11-Pad1) -> GND
- U5 pad 6: Net-(C9-Pad1) -> +VIN
- U6 pad 10: GND -> GPS_RST
- U6 pad 11: Net-(C9-Pad2) -> Net-(U6-Pad11)
- U6 pad 12: GND -> Net-(U6-Pad12)
- U6 pad 13: Net-(R11-Pad2) -> Net-(R3-Pad1)
- U6 pad 14: Net-(R12-Pad2) -> Net-(R10-Pad1)
- U6 pad 15: Net-(U6-Pad15) -> GND
- U6 pad 18: Net-(D1-Pad1) -> Net-(Q2-Pad2)
- U6 pad 2: GPS_TXD -> GND
- U6 pad 3: GPS_RXD -> GND
- U6 pad 4: GPS_PPS -> Net-(C10-Pad1)
- U6 pad 5: GPS_STDBY -> GND
- U6 pad 6: VCC -> Net-(C11-Pad1)
- U6 pad 7: Net-(U6-Pad7) -> GND
- U6 pad 8: Net-(C15-Pad1) -> +1.8V
- U6 pad 9: GPS_RST -> GND
- U9 pad 1: Net-(C15-Pad1) -> Net-(U6-Pad16)
- U9 pad 2: Net-(C15-Pad1) -> Net-(R3-Pad1)
- U9 pad 3: GND -> +1.8V
- U9 pad 5: VCC -> Net-(U6-Pad12)
- U9 pad 6: Net-(D1-Pad2) -> Net-(R10-Pad1)
- U9 pad 7: VCC -> +1.8V
- U9 pad 8: VCC -> +1.8V
Routing:
- net GND: track 116.8 -> 417.0 mm, vias 46 -> 121
- net VCC: track 59.1 -> 228.7 mm, vias 14 -> 19
- net +VIN: track 0.00 -> 99.8 mm, vias 0 -> 7
- net +1.8V: track 0.00 -> 72.1 mm, vias 0 -> 2
- net /MCU_DISPLAY/LCD_BKL2: track 0.00 -> 51.0 mm, vias 0 -> 3
- net BC_PGOOD_N: track 2.69 -> 32.2 mm, vias 2 -> 1
- net SD_EN: track 0.00 -> 29.0 mm, vias 0 -> 2
- net /MCU_DISPLAY/LCD_BKL1: track 0.00 -> 27.9 mm, vias 0 -> 5
- net /MCU_DISPLAY/SWDO: track 15.4 -> 42.7 mm, vias 0 -> 2
- net /MCU_DISPLAY/SWDIO: track 13.9 -> 40.9 mm, vias 0 -> 2
- net /MCU_DISPLAY/SWCLK: track 17.2 -> 42.6 mm, vias 0 -> 2
- net BC_CHG_N: track 2.70 -> 28.1 mm, vias 2 -> 1
- net SCL: track 38.8 -> 63.5 mm, vias 1 -> 5
- net Net-(C2-Pad1): track 22.5 -> 0.00 mm
- net Net-(R3-Pad1): track 0.00 -> 20.8 mm, vias 0 -> 2
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- added copper zone on Inner1.Cu, net +5V
- added copper zone on Inner1.Cu, net +VIN
- added copper zone on B.Cu, net GND
- added copper zone on F.Cu, net GND
- added copper zone on Inner2.Cu, net GND
- added copper zone on Inner1.Cu, net VCC
Other:
- outline, holes or cut-outs redrawn
- net class Default: via_dia 0.889 -> 1; via_drill 0.635 -> 0.5
- net class class3: via_dia 1.0668 -> 1; via_drill 0.6604 -> 0.5
- net class class4: via_dia 0.762 -> 0.75; via_drill 0.4572 -> 0.35
- net class class5: via_dia 0.762 -> 0.75; via_drill 0.4572 -> 0.35
- net class class6: via_dia 0.6096 -> 0.6; via_drill 0.3556 -> 0.25
- rule via_min_drill: 0.3556 -> 0.25
- rule via_min_size: 0.6096 -> 0.6
- board text added: "Freewatch v1.0"
- board text added: "Licensed under CERN OHL v.1.2"
- board text added: "Program/SWD"
